Commit message: add gazebo simulation pkg delta_amr2st_gazebo, update TY2_SW urdf model for gazebo, update gazebo world display

File: src/turtlebot3/turtlebot3_description/urdf/turtlebot3_burger.urdf.xacro (robot description, xacro)
@@ -31,5 +31,5 @@
     </inertial>
   </link>
-  <joint name="wheel_left_joint" type="continuous">
+  <joint name="wheel_left_joint" type="fixed">
     <parent link="base_link"/>
     <child link="wheel_left_link"/>
@@ -59,5 +59,5 @@
       </inertial>
   </link>
-  <joint name="wheel_right_joint" type="continuous">
+  <joint name="wheel_right_joint" type="fixed">
     <parent link="base_link"/>
     <child link="wheel_right_link"/>
