Commit message: complete TY2_SW.urdf

File: src/delta_amr2st_urdf/urdf/TY2_SW.urdf (robot description, URDF)
Before this commit: robot TY2_SW, 3 links, 2 joints
Links:
- added link body_link; visual box size=0.7 0.4 0.3
- added link realsensor_link; visual box size=0.05 0.16 0.05
- added link scanB_link; visual box size=0.14 0.14 0.08
- added link scanF_link; visual box size=0.14 0.14 0.08
- link Lwheel_link: mass 0.672830928354001 -> None; geometry visual cylinder length=0.04 radius=0.11
- link Rwheel_link: mass 0.672830928354001 -> None; geometry visual cylinder length=0.04 radius=0.11
- link base_link: mass 1.82224394008984 -> None
Joints:
- removed joint Lwheel_to_base
- removed joint Rwheel_to_base
- added joint base_to_Lwheel_joint: type fixed, parent base_link, child body_link, origin xyz=0 0 0.11 rpy=0 0 0
- added joint body_to_Lwheel_joint: type continuous, parent body_link, child Lwheel_link, origin xyz=0 0.2738 0 rpy=-1.5707 0 0, axis 0 1 0
- added joint body_to_Rwheel_joint: type continuous, parent body_link, child Rwheel_link, origin xyz=0 -0.2738 0 rpy=1.5707 0 0, axis 0 1 0
- added joint body_to_realsensor_joint: type fixed, parent body_link, child realsensor_link, origin xyz=0.4129 0 0.2675 rpy=0 0 0
- added joint body_to_scanB_joint: type fixed, parent body_link, child scanB_link, origin xyz=-0.33142 -0.22887 0.23138 rpy=0 0 3.1415926
- added joint body_to_scanF_joint: type fixed, parent body_link, child scanF_link, origin xyz=0.33142 0.22887 0.23138 rpy=0 0 0

Commit message: add simulation odometry function

File: src/delta_amr2st_urdf/urdf/TY2_SW.urdf (robot description, URDF)
Before this commit: robot TY2_SW, 7 links, 6 joints
Links:
- added link map_link
- added link odom_link
- link Lwheel_link: geometry visual cylinder length=0.05 radius=0.11
- link Rwheel_link: geometry visual cylinder length=0.05 radius=0.11
- link body_link: geometry visual box size=0.8 0.48 0.37
Joints:
- removed joint base_to_Lwheel_joint
- added joint base_to_body_joint: type fixed, parent base_link, child body_link, origin xyz=0 0 0 rpy=0 0 0
- added joint map_to_odom_joint: type fixed, parent map_link, child odom_link, origin xyz=0 0 0 rpy=0 0 0
- added joint odom_to_base_joint: type fixed, parent odom_link, child base_link, origin xyz=0 0 0.11 rpy=0 0 0
- joint body_to_scanB_joint: origin xyz=-0.33142 -0.22887 0.23138 rpy=0 0 3.1415926 -> xyz=-0.33142 0.22887 0.23138 rpy=0 0 2.3561944902
- joint body_to_scanF_joint: origin xyz=0.33142 0.22887 0.23138 rpy=0 0 0 -> xyz=0.33142 -0.22887 0.23138 rpy=0 0 -0.7853981634

Commit message: add odometry transform function and gmapping run test

File: src/delta_amr2st_urdf/urdf/TY2_SW.urdf (robot description, URDF)
Before this commit: robot TY2_SW, 9 links, 8 joints
Links:
- removed link map_link
- removed link odom_link
- added link map
- added link odom
Joints:
- joint map_to_odom_joint: child odom_link -> odom; parent map_link -> map
- joint odom_to_base_joint: parent odom_link -> odom

Commit message: add odometry and gmappingSLAM and hectorSLAM and imu-read-pkg

File: src/delta_amr2st_urdf/urdf/TY2_SW.urdf (robot description, URDF)
Before this commit: robot TY2_SW, 9 links, 8 joints
Links:
- added link imu_ch110_link; visual box size=0.04 0.4 0.025
Joints:
- added joint body_to_imu_joint: type fixed, parent body_link, child imu_ch110_link, origin xyz=0 0 -0.0246 rpy=0 0 0

Commit message: add mapping and move_base navigation function

File: src/delta_amr2st_urdf/urdf/TY2_SW.urdf (robot description, URDF)
Before this commit: robot TY2_SW, 10 links, 9 joints
Links:
- added link base_footprint
Joints:
- removed joint odom_to_base_joint
- added joint basefootprint_to_base_joint: type fixed, parent base_footprint, child base_link, origin xyz=0 0 0.11 rpy=0 0 0
- added joint odom_to_basefootprint_joint: type fixed, parent odom, child base_footprint, origin xyz=0 0 0 rpy=0 0 0

Commit message: add move_base param3, navigation complate using param1

File: src/delta_amr2st_urdf/urdf/TY2_SW.urdf (robot description, URDF)
Before this commit: robot TY2_SW, 11 links, 10 joints
Links:
- removed link map
- removed link odom
Joints:
- removed joint map_to_odom_joint
- removed joint odom_to_basefootprint_joint
- joint body_to_Lwheel_joint: type continuous -> fixed
- joint body_to_Rwheel_joint: type continuous -> fixed

Commit message: to do robot_pose_ekf

File: src/delta_amr2st_urdf/urdf/TY2_SW.urdf (robot description, URDF)
Before this commit: robot TY2_SW, 9 links, 8 joints
Links:
- added link lidarprom_link
Joints:
- added joint lidarprom_to_body_joint: type fixed, parent body_link, child lidarprom_link, origin xyz=0 0 0.25535 rpy=0 0 0
- joint body_to_scanB_joint: origin xyz=-0.33142 0.22887 0.23138 rpy=0 0 2.3561944902 -> xyz=-0.340895 0.2383385 0.25535 rpy=0 0 2.3561944902
- joint body_to_scanF_joint: origin xyz=0.33142 -0.22887 0.23138 rpy=0 0 -0.7853981634 -> xyz=0.340895 -0.2383385 0.25535 rpy=0 0 -0.7853981634

Commit message: robot_pose_ekf compile success, testing...

File: src/delta_amr2st_urdf/urdf/TY2_SW.urdf (robot description, URDF)
Before this commit: robot TY2_SW, 10 links, 9 joints
Links:
- removed link body_link
- link base_link: geometry visual box size=0.8 0.48 0.37
Joints:
- removed joint base_to_body_joint
- joint body_to_Lwheel_joint: parent body_link -> base_link
- joint body_to_Rwheel_joint: parent body_link -> base_link
- joint body_to_imu_joint: parent body_link -> base_link
- joint body_to_realsensor_joint: parent body_link -> base_link
- joint body_to_scanB_joint: parent body_link -> base_link
- joint body_to_scanF_joint: parent body_link -> base_link
- joint lidarprom_to_body_joint: parent body_link -> base_link

File: src/turtlebot3/turtlebot3_description/urdf/turtlebot3_burger.urdf.xacro (robot description, xacro)
@@ -31,5 +31,5 @@
     </inertial>
   </link>
-  <joint name="wheel_left_joint" type="fixed">
+  <joint name="wheel_left_joint" type="continuous">
     <parent link="base_link"/>
     <child link="wheel_left_link"/>
@@ -59,5 +59,5 @@
       </inertial>
   </link>
-  <joint name="wheel_right_joint" type="fixed">
+  <joint name="wheel_right_joint" type="continuous">
     <parent link="base_link"/>
     <child link="wheel_right_link"/>

Commit message: add send_goal.cpp

File: src/delta_amr2st_urdf/urdf/TY2_SW.urdf (robot description, URDF)
Before this commit: robot TY2_SW, 9 links, 8 joints
Links:
- removed link realsensor_link
- added link camera_link; visual box size=0.05 0.16 0.05
Joints:
- removed joint body_to_realsensor_joint
- added joint body_to_camera_joint: type fixed, parent base_link, child camera_link, origin xyz=0.4129 0.3 0.1 rpy=0 0 1.5707963268

Commit message: add tf_correction_update

File: src/delta_amr2st_urdf/urdf/TY2_SW.urdf (robot description, URDF)
Before this commit: robot TY2_SW, 9 links, 8 joints
Joints:
- joint body_to_camera_joint: origin xyz=0.4129 0.3 0.1 rpy=0 0 1.5707963268 -> xyz=0.5 0.0 0.1 rpy=0 0 3.1415926536
